File: boards/lite/kicad/lite-main.kicad_sch (KiCad schematic)
At the start: 130 parts, among them J1 USB4105-GF-A-120, J2 RCA line in, J3 RCA sub out, J4 DB128V-5.08-4P, Q1 AO4485, Q2 MMBT3904, Q3 MMBT3904, Q4 MMBT3904, SW1 TS-1187A, SW2 TS-1187A, SW3 TS-1187A, U1 CH224A, U2 TPS54302, U3 SY8089A1AAC, U4 LP5907-3.3, U5 ESP32-WROVER-E-N8R8, U6 CH340C, U7 ES8388, U8 TPA3118D2, U9 IRM-H638T

Commit message: lite-main: routed, drc_routed 0/0; front-facing IR receiver, PVDD sense on GPIO39
Parts:
- added C18: 100nF, Capacitor_SMD:C_0603_1608Metric, symbol Device:C
- added R17: 100k, Resistor_SMD:R_0603_1608Metric, symbol Device:R
- added R18: 10k, Resistor_SMD:R_0603_1608Metric, symbol Device:R
- added R65: 100R, Resistor_SMD:R_0603_1608Metric, symbol Device:R
- C80: value 100nF -> 4.7uF; LCSC C14663 -> C19666
- U9: value IRM-H638T -> IRM-3638T; footprint aiee:SENSOR-SMD_IRM-H638T-TR2-TL -> aiee:OPTO-TH_IRM-3638T; symbol aiee:IRM-H638T_TR2 -> aiee:IRM-3638T_C42421366; LCSC C91447 -> C42421366
Connections:
- net +3V3: now also R65.1; no longer C80.1, U9.4 (VCC)
- net GND: now also C18.2, R18.2; no longer U9.1 (GND)
- net IR_IN: now also U9.1 (OUT); no longer U9.3 (VOUT)
- net PVDD: now also R17.1
- net PVDD_SENSE: now reaches U5.5 (SENSOR_VN)
- net PVDD_SENSE: now also C18.1, R17.2, R18.1
- new net IR_VCC: C80.1, R65.2, U9.3 (VCC)
- no-connect marks 32 -> 31
Other:
- moved on the sheet: C80, D2, R63, R64
