File: boards/lite/kicad/lite-main.kicad_pcb (KiCad board)
At the start: 2 copper layers, 100 x 90 mm, 138 parts, among them J1 USB4105-GF-A-120, J2 RCA line in, J3 RCA sub out, J4 DB128V-5.08-4P, Q1 AO4485, Q2 MMBT3904, Q3 MMBT3904, Q4 MMBT3904, SW1 TS-1187A, SW2 TS-1187A, SW3 TS-1187A, U1 CH224A, U2 TPS54302, U3 SY8089A1AAC, U4 LP5907-3.3, U5 ESP32-WROVER-E-N8R8, U6 CH340C, U7 ES8388, U8 TPA3118D2, U9 IRM-3638T

Commit message: lite-main: board review fixes (TVS at the VBUS pour, U3 input loop on top, EP paste windows, J4 polarity silk); re-routed; all gates pass
Parts:
- moved D1 8.16 mm to (84.9, 72.2), turned to 180 degrees
- moved C11 6.19 mm to (74.9, 99.7), turned to 0 degrees
- moved C10 4.88 mm to (74.9, 97.9), turned to 0 degrees
- moved R7 4.00 mm to (83.4, 77.0)
- moved Q4 3.80 mm to (86.9, 75.9)
Routing:
- net +3V3: track 313.0 -> 264.9 mm
- net /VBUS_SENSE: track 65.0 -> 48.3 mm
- net /I2C_SCL: track 109.9 -> 96.0 mm, vias 5 -> 4
- net /PVDD_EN: track 74.9 -> 87.8 mm
- net GND: track 149.5 -> 162.1 mm, vias 109 -> 115
- net /AMP_IN_R: track 65.1 -> 75.4 mm
- net /BUCK3_LX: track 4.36 -> 13.8 mm
- net /I2C_SDA: track 110.5 -> 119.7 mm, vias 4 -> 5
- net /AMP_IN_L: track 51.2 -> 60.0 mm, vias 2 -> 4
- net /USB_DP: track 65.1 -> 73.1 mm
- net /USB_DM: track 63.4 -> 71.4 mm
- net /PD_PG: track 87.7 -> 95.3 mm
- net /LINEIN_L: track 17.4 -> 23.8 mm
- net /PSW_PULL: track 10.4 -> 5.48 mm
- net /AMP_SDZ_IO: track 70.7 -> 65.9 mm
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Other:
- board text added: "L+"
- board text added: "L-"
- board text added: "R+"
- board text added: "R-"
