File: boards/core/kicad/core.kicad_pcb (KiCad board)
At the start: 4 copper layers, 120 x 100 mm, 301 parts, among them J1 USB4085-GF-A, J10 SPK B L, J11 SPK B R, J2 HR911105A, J3 FFC 20P, J4 SUB OUT, J5 LINE IN, J6 SPK A L, J7 SPK A R, Q1 AO4485, Q2 2N7002, Q3 S8050, Q4 S8050, Q5 S8050, Q6 S8050, Q7 S8050, SW1 EC11, SW2 BTN1, SW3 BTN2, U1 CH224Q, U10 ES9018K2M, U11 OPA1678, U12 PCM5102A, U13 ES7243E, U14 TS5A23157, U15 TPA3221, U16 TPA3221, U17 TCA9539, U18 IRM-3638T, U19 PLR237/T8BK, U2 USBLC6-2SC6, U20 TS5A23157, U3 INA186A1, U4 SY8303AIC, U5 SY8089A1AAC, U6 LP5907-3.3, U7 ESP32-WROVER-E-N8R8, U8 CH340B, U9 LAN8720A, Y1 49.152MHz, Y2 50MHz

Commit message: First-spin review: every finding's disposition, known-unknowns resolved for Lite and Plus (order gate by tier), firmware duties for core, R45 2.2k, honest TPA3221 thermal constraint, Plus/Ultra cost estimate
Parts:
- R45: value 10k -> 2.2k
Changed lines of the file:
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@@
 			)
 		)
-		(property "Value" "10k"
+		(property "Value" "2.2k"
 			(at 0 4 0)
 			(layer "F.Fab")
@@
 			)
 		)
-		(property "LCSC" "C25744"
+		(property "LCSC" "C25879"
 			(at 0 0 0)
 			(layer "F.SilkS")
