File: boards/core/kicad/core.kicad_pcb (KiCad board)
At the start: 4 copper layers, 120 x 100 mm, 282 parts, among them J1 USB4105-GF-A-120, J10 SPK B L, J11 SPK B R, J2 HR911105A, J3 FFC 20P, J4 SUB OUT, J5 LINE IN, J6 SPK A L, J7 SPK A R, Q1 AO4485, Q2 2N7002, Q3 S8050, Q4 S8050, Q5 S8050, Q6 S8050, SW1 EC11, SW2 BTN1, SW3 BTN2, U1 CH224Q, U10 ES9018K2M, U11 OPA1678, U12 PCM5102A, U13 ES7243E, U14 TS5A23157, U15 TPA3221, U16 TPA3221, U17 TCA9555, U18 IRM-H638T, U19 PLR237/T8BK, U2 USBLC6-2SC6, U3 INA186A1, U4 SY8303AIC, U5 SY8089A1AAC, U6 LP5907-3.3, U7 ESP32-WROVER-E-N8R8, U8 CH340C, U9 LAN8720A, Y1 50MHz, Y2 50MHz

Commit message: core carries its real 5 A VBUS/PVDD current in every layer's pour, and +5V's trunk layer changes get two vias
Budgets at real currents (VBUS_IN/VBUS/PVDD 5 A, +5V 0.65 A); check_current
passes with each layer's pour judged alone. In1/In2 to 1 oz; kicad/gen/power_trunk.py
clears the GND stitch grid from the In2 power planes, reshapes their zones, moves
three vias, gives each PVDD finger five plane vias and +5V's trunk two vias per
layer change. Gerbers regenerated.
Routing:
- net PVDD: track 79.4 -> 70.8 mm, vias 23 -> 34
- net +5V: track 262.2 -> 265.5 mm, vias 6 -> 8
- net GND: track 53.5 -> 54.2 mm, vias 261 -> 182
