File: boards/core/kicad/core.kicad_pcb (KiCad board)
At the start: 4 copper layers, 154.4 x 113 mm, 312 parts, among them J1 USB4085-GF-A, J2 HR911105A, J20 24.243 red, J21 24.243 black, J22 24.243 red, J23 24.243 black, J24 24.243 red, J25 24.243 black, J26 24.243 red, J27 24.243 black, J3 FFC 20P, J4 SUB OUT, J5 LINE IN, Q1 AO4485, Q2 2N7002, Q3 MMDT3904, Q4 S8050, Q5 S8050, Q6 S8050, Q7 S8050, SW1 EC11, SW2 BTN1, SW3 BTN2, U1 CH224Q, U10 ES9018K2M, U11 OPA1678, U12 PCM5102A, U13 ES7243E, U14 TS5A23157, U15 TPA3220, U16 TPA3220, U17 TCA9539, U18 IRM-3638T, U19 PLR237/T8BK, U2 USBLC6-2SC6, U20 TS5A23157, U21 TLV803S, U3 INA186A1, U4 SY8303AIC, U5 SY8089A1AAC, U6 LP5907-3.3, U7 ESP32-WROVER-E-N8R8, U8 CH340B, U9 LAN8720A, Y1 49.152MHz, Y2 50MHz

Commit message: WIP core banana: speaker pours as one staircase polygon per net, In2 pin links, C4/C8 (R5-PA-1), DAL-7, stubs ripped
Parts:
- C4: value 100nF -> 220nF
- C8: value 2.2uF -> 4.7uF
Routing:
- net /linein/LIN_L: track 16.1 -> 0.00 mm, vias 1 -> 0
- net /amp_b/B_SPK_L-: track 8.71 -> 24.4 mm
- net /amp_b/B_SPK_L+: track 3.97 -> 18.3 mm
- net /amp_a/A_SPK_R-: track 5.60 -> 18.2 mm
- net /OPT_SPDIF: track 11.8 -> 0.00 mm, vias 1 -> 0
- net /linein/LIN_R: track 12.0 -> 1.45 mm, vias 1 -> 0
- net /A_SPK_L+: track 59.7 -> 56.3 mm
- net /A_SPK_R+: track 43.4 -> 40.2 mm, vias 1 -> 0
- net /amp_b/B_SPK_R-: track 5.60 -> 2.48 mm
- net /dac/SUB2_OUT: track 5.56 -> 4.67 mm, vias 1 -> 0
- net /dac/SUB1_OUT: vias 1 -> 0
