File: boards/core/kicad/mcu.kicad_sch (KiCad schematic)
At the start: 35 parts, among them Q4 S8050, Q5 S8050, U17 TCA9555, U7 ESP32-WROVER-E-N8R8, U8 CH340C

Commit message: core (Plus/Ultra) after the first-spin review: TCA9539 with ESP32 reset, 5 A path via patches and through-hole USB4085, antenna keep-out, PVDD switch SOA and PD-PG gating, OPA1678 headroom, RCA and TOSLINK holes, front IR, 49.152 MHz DAC clock, speaker loopback taps; all gates pass
Review-2 blockers fixed on core: DIGITAL-1/2/PARTS-4, POWER-1, DFM-1, PARTS-7;
THERMAL-1 handled by a lid-pressed heatsink plus firmware governor (no room
for clip holes). Majors: POWER-2/6, AUDIO-1/2/3, DIGITAL-19, DFM-4. Done as an
ECO on the routed board; Ultra zone-B taps left out (no control line).
Parts:
- R45: value 100k -> 10k; LCSC C25741 -> C25744
- U17: value TCA9555 -> TCA9539; symbol aiee:TCA9555PWR -> aiee:TCA9539PWR; LCSC C465732 -> C131972
- U8: value CH340C -> CH340B; symbol aiee:CH340C -> aiee:CH340B; LCSC C84681 -> C81010
Connections:
- net +3V3: no longer R57.1
- net ESP_EN: now also U17.3 (~{RESET})
- net GND: now also R57.2; no longer U17.3 (A2)
- net LCD_CS: now also R57.1; no longer R57.2, U17.20 (P17)
- new net TAP_SEL_IO: U17.20 (P17)
Other:
- moved on the sheet: C30, C31, C32, C33, C34, C37, C38, C39, Q4, Q5, R30, R31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

Commit message: First-spin review: every finding's disposition, known-unknowns resolved for Lite and Plus (order gate by tier), firmware duties for core, R45 2.2k, honest TPA3221 thermal constraint, Plus/Ultra cost estimate
Parts:
- R45: value 10k -> 2.2k; LCSC C25744 -> C25879
Changed lines of the file:
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@@
 			)
 		)
-		(property "Value" "10k"
+		(property "Value" "2.2k"
 			(at 162.306 224.79 0.0000)
 			(effects
@@
 			)
 		)
-		(property "LCSC" "C25744"
+		(property "LCSC" "C25879"
 			(at 162.56 228.5999 0)
 			(effects
