File: boards/core/kicad/mcu.kicad_sch (KiCad schematic)
At the start: 35 parts, among them Q4 S8050, Q5 S8050, U17 TCA9555, U7 ESP32-WROVER-E-N8R8, U8 CH340C

Commit message: The boards will work on the first spin: independent engineering reviews of Lite and core, fixes and contingencies built…
* First-spin review: the brief each domain reviewer works from

* First-spin review: partial drafts saved before the reviewers' login d…

…ropped

* First-spin review: power, audio, digital and thermal reviews of lite-…

…main and core, with their sims

* core carries its EasyEDA CPL model cache, so its dfm gate runs withou…

…t EasyEDA (red on 403 otherwise); DFM review

* First-spin review: parts pin-to-pad audit of both boards

* Lite board after the first-spin review: amp SDZ, PVDD switch hold-off…

… and soft start, line-in headroom, 5 V loop, RCA slots, HRO USB-C and CH340B, speaker loopback taps; regenerated on hwde c23e27e, all gates pass

Review-2 findings fixed on lite-main as an ECO on the routed board (no
re-route): AUDIO-4/DIGITAL-14, POWER-3/4/10, AUDIO-7, DFM-2, stock swaps.
Also: the speaker loopback taps (task 261029-033806) and the hwde refresh
(task 261029-004401) for this board. Known-unknowns list and its order-step
check (tools/known_unknowns.py). Unit cost at 100: 13.16 (was 13.05).

* core (Plus/Ultra) after the first-spin review: TCA9539 with ESP32 res…

…et, 5 A path via patches and through-hole USB4085, antenna keep-out, PVDD switch SOA and PD-PG gating, OPA1678 headroom, RCA and TOSLINK holes, front IR, 49.152 MHz DAC clock, speaker loopback taps; all gates pass

Review-2 blockers fixed on core: DIGITAL-1/2/PARTS-4, POWER-1, DFM-1, PARTS-7;
THERMAL-1 handled by a lid-pressed heatsink plus firmware governor (no room
for clip holes). Majors: POWER-2/6, AUDIO-1/2/3, DIGITAL-19, DFM-4. Done as an
ECO on the routed board; Ultra zone-B taps left out (no control line).

* First-spin review: every finding's disposition, known-unknowns resolv…

…ed for Lite and Plus (order gate by tier), firmware duties for core, R45 2.2k, honest TPA3221 thermal constraint, Plus/Ultra cost estimate

* Heatsink options for the TPA3221 checked aga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
Parts:
- R45: value 100k -> 2.2k; LCSC C25741 -> C25879
- U17: value TCA9555 -> TCA9539; symbol aiee:TCA9555PWR -> aiee:TCA9539PWR; LCSC C465732 -> C131972
- U8: value CH340C -> CH340B; symbol aiee:CH340C -> aiee:CH340B; LCSC C84681 -> C81010
Connections:
- net +3V3: no longer R57.1
- net ESP_EN: now also U17.3 (~{RESET})
- net GND: now also R57.2; no longer U17.3 (A2)
- net LCD_CS: now also R57.1; no longer R57.2, U17.20 (P17)
- new net TAP_SEL_IO: U17.20 (P17)
Other:
- moved on the sheet: C30, C31, C32, C33, C34, C37, C38, C39, Q4, Q5, R30, R31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

Commit message: core: a 2.93 V supervisor (TLV803S) on ESP_EN, so a brownout resets the expander and the PHY clock with the ESP32 (R3-DIGITAL-1); VREF's C64 10 uF -> 100 uF 1206 (R3-AUDIO-1)
U21 sits by R30 and joins ESP_EN and +3V3; C64 moved to the free spot beside
R73 and rejoined to VREF. Prices kept from the committed parts.json; the two
new lines priced live (tools/price_parts.py). DRC clean, zones refilled.
Parts:
- added U21: TLV803S, aiee:SOT-23-3_L2.9-W1.3-P1.90-LS2.4-BR, symbol aiee:TLV803SDBZR
Connections:
- net +3V3: now also U21.3 (VDD)
- net ESP_EN: now also U21.2 (~{RESET})
- net GND: now also U21.1 (GND)
Other:
- moved on the sheet: C30, C31, C32, C33, C34, C37, C38, C39, Q4, Q5, R30, R31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
