File: boards/core/kicad/amp_b.kicad_sch (KiCad schematic)
At the start: 42 parts, among them J10 SPK B L, J11 SPK B R, U16 TPA3221

Commit message: Plus/Ultra amps need no hand-fitted heatsink: U15/U16 are the pin-identical pad-down TPA3220, EP soldered to the GND planes
No JLC process fits a heatsink onto the TPA3221's top slug (LCSC's pinned heatsinks are TO-220 extrusions, and none fits the 19x12 mm room), so core takes TI's pad-down twin, the TPA3220DDW (SLASEN3B table 5: pin-compatible). It gets a new symbol (+pin 45 EP) and a footprint with a 7.3x4.43 EP, 15 x 0.3 mm vias and 4 paste windows. The footprint was swapped in place, the copper under the body ripped and re-routed with route_finish, and DRC, verify, dfm and erc all pass. The fab package for Plus and Ultra is regenerated, with the C2879306 EasyEDA cache.

Thermal (~26 C/W into the board): 1/8 power into 8 ohm holds (Tj ~84 C). Into 4 ohm the firmware governor holds the chip near 2.4 W (16 W in, 60 s), with 77 W peaks kept. Constraints, firmware-requirements C2/C3, product.md, the README/blocks docs, the manual, bom-estimate/bom-stock, the known-unknowns resolutions and heatsink-options.md all match.

LCSC/JLC stock 0: buy it into the JLC inventory (Mouser 6,566, DigiKey 2,032); see fab/prebuy.csv.
Parts:
- U16: value TPA3221 -> TPA3220; footprint aiee:HTSSOP-44_L14.0-W6.1-P0.64-LS8.1-BL -> aiee:HTSSOP-44-1EP_L14.0-W6.1-P0.64-LS8.1-EP7.3x4.43; symbol aiee:TPA3221DDVR -> aiee:TPA3220DDWR; LCSC C475500 -> C2879306
Connections:
- net GND: now also U16.45 (GND)
Other:
- moved on the sheet: C301, C302, C304, C306, C307, C308, C309, C310, C311, C312, C316, C317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

Commit message: Plus keeps its power: both TPA3220s fitted, L on zone A and R on zone B (one channel per chip), firmware HIFI_SPLIT and a 10 W governor; loud-music thermal table from hwde check_thermal; the trade-off in product.md
Parts:
- C301, C302, C304, C306, C307, C308, C309, C310, C311, C312, C316, C317, C318, C319, C320, C321, C322, C323, C324, C326, C327, C329, C330, C332, C333, C335, J10, J11, L5, L6, L7, L8, R303, R305, R313, R314, R315, R325, R328, R331, R334, U16: now fitted
Changed lines of the file:
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@@
 		(in_bom yes)
 		(on_board yes)
-		(dnp yes)
+		(dnp no)
 		(fields_autoplaced no)
 		(property "Reference" "U16"
@@
 		(in_bom yes)
 		(on_board yes)
-		(dnp yes)
+		(dnp no)
 		(fields_autoplaced no)
 		(property "Reference" "C301"
@@
 		(in_bom yes)
 		(on_board yes)
-		(dnp yes)
+		(dnp no)
 		(fields_autoplaced no)
 		(property "Reference" "C302"
@@
 		(in_bom yes)
 		(on_board yes)
-		(dnp yes)
+		(dnp no)
 		(fields_autoplaced no)
 		(property "Reference" "R303"
@@
 		(in_bom yes)
 		(on_board yes)
-		(dnp yes)
+		(dnp no)
 		(fields_autoplaced no)
 		(property "Reference" "C304"
@@
 		(in_bom yes)
 		(on_board yes)
-		(dnp yes)
+		(dnp no)
 		(fields_autoplaced no)
 		(property "Reference" "R305"
@@
 		(in_bom yes)
 		(on_board yes)
-		(dnp yes)
+		(dnp no)
 		(fields_autoplaced no)
 		(property "Reference" "C306"
@@
 		(in_bom yes)
 		(on_board yes)
-		(dnp yes)
+		(dnp no)
 		(fields_autoplaced no)
 		(property "Reference" "C307"
@@
 		(in_bom yes)
 		(on_board yes)
-		(dnp yes)
+		(dnp no)
 		(fields_autoplaced no)
 		(property "Reference" "C308"
@@
 		(in_bom yes)
 		(on_board yes)
-		(dnp yes)
+		(dnp no)
 		(fields_autoplaced no)
 		(property "Reference" "C309"
@@
 		(in_bom yes)
 		(on_board yes)
-		(dnp yes)
+		(dnp no)
 		(fields_autoplaced no)
 		(property "Reference" "C310"
@@
 		(in_bom yes)
 		(on_board yes)
-		(dnp yes)
+		(dnp no)
 		(fields_autoplaced no)
 		(property "Reference" "C311"
@@
 		(in_bom yes)
 		(on_board yes)
-		(dnp yes)
+		(dnp no)
 		(fields_autoplaced no)
 		(property "Reference" "C312"
@@
 		(in_bom yes)
 		(on_board yes)
-		(dnp yes)
+		(dnp no)
 		(fields_autoplaced no)
 		(property "Reference" "R313"
@@
 		(in_bom yes)
 		(on_board yes)
-		(dnp yes)
+		(dnp no)
 		(fields_autoplaced no)
 		(property "Reference" "R314"
@@
 		(in_bom yes)
 		(on_board yes)
-		(dnp yes)
+		(dnp no)
 		(fields_autoplaced no)
 		(property "Reference" "R315"
@@
 		(in_bom yes)
 		(on_board yes)
-		(dnp yes)
+		(dnp no)
 		(fields_autoplaced no)
 		(property "Reference" "C316"
@@
 		(in_bom yes)
 		(on_board yes)
-		(dnp yes)
+		(dnp no)
 		(fields_autoplaced no)
 		(property "Reference" "C317"
@@
 		(in_bom yes)
 		(on_board yes)
-		(dnp yes)
+		(dnp no)
 		(fields_autoplaced no)
 		(property "Reference" "C318"
@@
 		(in_bom yes)
 		(on_board yes)
-		(dnp yes)
+		(dnp no)
 		(fields_autoplaced no)
 		(property "Reference" "C319"
@@
 		(in_bom yes)
 		(on_board yes)
-		(dnp yes)
+		(dnp no)
 		(fields_autoplaced no)
 		(property "Reference" "C320"
@@
 		(in_bom yes)
 		(on_board yes)
-		(dnp yes)
+		(dnp no)
 		(fields_autoplaced no)
 		(property "Reference" "C321"
@@
 		(in_bom yes)
 		(on_board yes)
-		(dnp yes)
+		(dnp no)
 		(fields_autoplaced no)
 		(property "Reference" "C322"
@@
 		(in_bom yes)
 		(on_board yes)
-		(dnp yes)
+		(dnp no)
 		(fields_autoplaced no)
 		(property "Reference" "C323"
@@
 		(in_bom yes)
 		(on_board yes)
-		(dnp yes)
+		(dnp no)
 		(fields_autoplaced no)
 		(property "Reference" "L5"
@@
 		(in_bom yes)
 		(on_board yes)
-		(dnp yes)
+		(dnp no)
 		(fields_autoplaced no)
 		(property "Reference" "C324"
@@
 		(in_bom yes)
 		(on_board yes)
-		(dnp yes)
+		(dnp no)
 		(fields_autoplaced no)
 		(property "Reference" "R325"
@@
 		(in_bom yes)
 		(on_board yes)
-		(dnp yes)
+		(dnp no)
 		(fields_autoplaced no)
 		(property "Reference" "C326"
@@
 		(in_bom yes)
 		(on_board yes)
-		(dnp yes)
+		(dnp no)
 		(fields_autoplaced no)
 		(property "Reference" "L6"
@@
 		(in_bom yes)
 		(on_board yes)
-		(dnp yes)
+		(dnp no)
 		(fields_autoplaced no)
 		(property "Reference" "C327"
@@
 		(in_bom yes)
 		(on_board yes)
-		(dnp yes)
+		(dnp no)
 		(fields_autoplaced no)
 		(property "Reference" "R328"
@@
 		(in_bom yes)
 		(on_board yes)
-		(dnp yes)
+		(dnp no)
 		(fields_autoplaced no)
 		(property "Reference" "C329"
@@
 		(in_bom yes)
 		(on_board yes)
-		(dnp yes)
+		(dnp no)
 		(fields_autoplaced no)
 		(property "Reference" "L7"
@@
 		(in_bom yes)
 		(on_board yes)
-		(dnp yes)
+		(dnp no)
 		(fields_autoplaced no)
 		(property "Reference" "C330"
@@
 		(in_bom yes)
 		(on_board yes)
-		(dnp yes)
+		(dnp no)
 		(fields_autoplaced no)
 		(property "Reference" "R331"
@@
 		(in_bom yes)
 		(on_board yes)
-		(dnp yes)
+		(dnp no)
 		(fields_autoplaced no)
 		(property "Reference" "C332"
@@
 		(in_bom yes)
 		(on_board yes)
-		(dnp yes)
+		(dnp no)
 		(fields_autoplaced no)
 		(property "Reference" "L8"
@@
 		(in_bom yes)
 		(on_board yes)
-		(dnp yes)
+		(dnp no)
 		(fields_autoplaced no)
 		(property "Reference" "C333"
@@
 		(in_bom yes)
 		(on_board yes)
-		(dnp yes)
+		(dnp no)
 		(fields_autoplaced no)
 		(property "Reference" "R334"
@@
 		(in_bom yes)
 		(on_board yes)
-		(dnp yes)
+		(dnp no)
 		(fields_autoplaced no)
 		(property "Reference" "C335"
@@
 		(in_bom yes)
 		(on_board yes)
-		(dnp yes)
+		(dnp no)
 		(fields_autoplaced no)
 		(property "Reference" "J10"
@@
 		(in_bom yes)
 		(on_board yes)
-		(dnp yes)
+		(dnp no)
 		(fields_autoplaced no)
 		(property "Reference" "J11"
