File: boards/core/kicad/amp_b.kicad_sch (KiCad schematic)
At the start: 42 parts, among them J10 SPK B L, J11 SPK B R, U16 TPA3221

Commit message: The boards will work on the first spin: independent engineering reviews of Lite and core, fixes and contingencies built…
* First-spin review: the brief each domain reviewer works from

* First-spin review: partial drafts saved before the reviewers' login d…

…ropped

* First-spin review: power, audio, digital and thermal reviews of lite-…

…main and core, with their sims

* core carries its EasyEDA CPL model cache, so its dfm gate runs withou…

…t EasyEDA (red on 403 otherwise); DFM review

* First-spin review: parts pin-to-pad audit of both boards

* Lite board after the first-spin review: amp SDZ, PVDD switch hold-off…

… and soft start, line-in headroom, 5 V loop, RCA slots, HRO USB-C and CH340B, speaker loopback taps; regenerated on hwde c23e27e, all gates pass

Review-2 findings fixed on lite-main as an ECO on the routed board (no
re-route): AUDIO-4/DIGITAL-14, POWER-3/4/10, AUDIO-7, DFM-2, stock swaps.
Also: the speaker loopback taps (task 261029-033806) and the hwde refresh
(task 261029-004401) for this board. Known-unknowns list and its order-step
check (tools/known_unknowns.py). Unit cost at 100: 13.16 (was 13.05).

* core (Plus/Ultra) after the first-spin review: TCA9539 with ESP32 res…

…et, 5 A path via patches and through-hole USB4085, antenna keep-out, PVDD switch SOA and PD-PG gating, OPA1678 headroom, RCA and TOSLINK holes, front IR, 49.152 MHz DAC clock, speaker loopback taps; all gates pass

Review-2 blockers fixed on core: DIGITAL-1/2/PARTS-4, POWER-1, DFM-1, PARTS-7;
THERMAL-1 handled by a lid-pressed heatsink plus firmware governor (no room
for clip holes). Majors: POWER-2/6, AUDIO-1/2/3, DIGITAL-19, DFM-4. Done as an
ECO on the routed board; Ultra zone-B taps left out (no control line).

* First-spin review: every finding's disposition, known-unknowns resolv…

…ed for Lite and Plus (order gate by tier), firmware duties for core, R45 2.2k, honest TPA3221 thermal constraint, Plus/Ultra cost estimate

* Heatsink options for the TPA3221 checked aga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
Parts:
- J10, J11: MPN (none) -> KF301-5.0-2P
Other:
- moved on the sheet: C301, C302, C304, C306, C307, C308, C309, C310, C311, C312, C316, C317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

Commit message: TPA3221 heatsink the person doesn't have to fit: a JLC-fittable board-mount part or a pad-down amp
* First-spin review: the brief each domain reviewer works from

* First-spin review: partial drafts saved before the reviewers' login d…

…ropped

* First-spin review: power, audio, digital and thermal reviews of lite-…

…main and core, with their sims

* core carries its EasyEDA CPL model cache, so its dfm gate runs withou…

…t EasyEDA (red on 403 otherwise); DFM review

* First-spin review: parts pin-to-pad audit of both boards

* Lite board after the first-spin review: amp SDZ, PVDD switch hold-off…

… and soft start, line-in headroom, 5 V loop, RCA slots, HRO USB-C and CH340B, speaker loopback taps; regenerated on hwde c23e27e, all gates pass

Review-2 findings fixed on lite-main as an ECO on the routed board (no
re-route): AUDIO-4/DIGITAL-14, POWER-3/4/10, AUDIO-7, DFM-2, stock swaps.
Also: the speaker loopback taps (task 261029-033806) and the hwde refresh
(task 261029-004401) for this board. Known-unknowns list and its order-step
check (tools/known_unknowns.py). Unit cost at 100: 13.16 (was 13.05).

* core (Plus/Ultra) after the first-spin review: TCA9539 with ESP32 res…

…et, 5 A path via patches and through-hole USB4085, antenna keep-out, PVDD switch SOA and PD-PG gating, OPA1678 headroom, RCA and TOSLINK holes, front IR, 49.152 MHz DAC clock, speaker loopback taps; all gates pass

Review-2 blockers fixed on core: DIGITAL-1/2/PARTS-4, POWER-1, DFM-1, PARTS-7;
THERMAL-1 handled by a lid-pressed heatsink plus firmware governor (no room
for clip holes). Majors: POWER-2/6, AUDIO-1/2/3, DIGITAL-19, DFM-4. Done as an
ECO on the routed board; Ultra zone-B taps left out (no control line).

* First-spin review: every finding's disposition, known-unknowns resolv…

…ed for Lite and Plus (order gate by tier), firmware duties for core, R45 2.2k, honest TPA3221 thermal constraint, Plus/Ultra cost estimate

* Heatsink options for the TPA3221 checked against the lead's order;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
Parts:
- C301, C302, C304, C306, C307, C308, C309, C310, C311, C312, C316, C317, C318, C319, C320, C321, C322, C323, C324, C326, C327, C329, C330, C332, C333, C335, J10, J11, L5, L6, L7, L8, R303, R305, R313, R314, R315, R325, R328, R331, R334: now fitted
- U16: value TPA3221 -> TPA3220; footprint aiee:HTSSOP-44_L14.0-W6.1-P0.64-LS8.1-BL -> aiee:HTSSOP-44-1EP_L14.0-W6.1-P0.64-LS8.1-EP7.3x4.43; symbol aiee:TPA3221DDVR -> aiee:TPA3220DDWR; LCSC C475500 -> C2879306; now fitted
Connections:
- net GND: now also U16.45 (GND)

Commit message: core amp-area ECO (#121): TPA3220 PVDD HF pairs under the pins and BST caps at the row ends (R3-AMP-1/2), U15's input caps at the IN pins (R3-LAYOUT-1); two-sided build, every gate passes
Parts:
- C307, C309: footprint aiee:C0805 -> aiee:C1206; LCSC C28323 -> C282823
Changed lines of the file:
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@@
 			)
 		)
-		(property "Footprint" "aiee:C0805"
+		(property "Footprint" "aiee:C1206"
 			(at 274.0152 148.59 0.0000)
 			(effects
@@
 			)
 		)
-		(property "LCSC" "C28323"
+		(property "LCSC" "C282823"
 			(at 275.59 157.4799 0)
 			(effects
@@
 			)
 		)
-		(property "Footprint" "aiee:C0805"
+		(property "Footprint" "aiee:C1206"
 			(at 309.5752 148.59 0.0000)
 			(effects
@@
 			)
 		)
-		(property "LCSC" "C28323"
+		(property "LCSC" "C282823"
 			(at 311.15 157.4799 0)
 			(effects
