File: boards/core/kicad/amp_b.kicad_sch (KiCad schematic)
At the start: 42 parts, among them J10 SPK B L, J11 SPK B R, U16 TPA3220

Commit message: Revert "core amp-area layout ECO: TPA3220 bootstrap and PVDD HF caps at their pins, input caps at the IN pins"
This reverts commit f0eb13530c5fd08d8df6501fd36629fa8401f02f.
Parts:
- C307, C309: footprint aiee:C1206 -> aiee:C0805; LCSC C282823 -> C28323
Changed lines of the file:
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@@
 			)
 		)
-		(property "Footprint" "aiee:C1206"
+		(property "Footprint" "aiee:C0805"
 			(at 274.0152 148.59 0.0000)
 			(effects
@@
 			)
 		)
-		(property "LCSC" "C282823"
+		(property "LCSC" "C28323"
 			(at 275.59 157.4799 0)
 			(effects
@@
 			)
 		)
-		(property "Footprint" "aiee:C1206"
+		(property "Footprint" "aiee:C0805"
 			(at 309.5752 148.59 0.0000)
 			(effects
@@
 			)
 		)
-		(property "LCSC" "C282823"
+		(property "LCSC" "C28323"
 			(at 311.15 157.4799 0)
 			(effects
