File: boards/core/kicad/amp_b.kicad_sch (KiCad schematic)
At the start: 42 parts, among them J10 SPK B L, J11 SPK B R, U16 TPA3220

Commit message: core's class-D outputs are damped with no speaker: the 4.7R snubbers get 470nF Zobel caps (#137)
The 8 per-leg snubber caps C228/C231/C234/C237/C326/C329/C332/C335 go from
1nF to 470nF/50V X7R 0603 (Yageo CC0603KRX7R9BB474, LCSC C513577). Same
footprints: board_update changed only value and LCSC fields, no copper.
Open-load peak +39.7 dB -> +15.8 dB (ngspice, docs/boards/sims/zobel_sweep.py);
4/6/8 ohm responses move under 0.6 dB. Test tones refuse a sine above 5 kHz
louder than -16 dBFS without force, so the 0603 resistors stay in rating.
Lite checked the same way and left as it is (docs/boards/core-zobel.md).

Co-Authored-By: Claude Opus 5.5 <noreply@anthropic.com>
Parts:
- C326, C329, C332, C335: value 1nF -> 470nF; LCSC C1588 -> C513577
Changed lines of the file:
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@@
 			)
 		)
-		(property "Value" "1nF"
+		(property "Value" "470nF"
 			(at 178.562 232.41 0.0000)
 			(effects
@@
 			)
 		)
-		(property "LCSC" "C1588"
+		(property "LCSC" "C513577"
 			(at 177.8 236.2199 0)
 			(effects
@@
 			)
 		)
-		(property "Value" "1nF"
+		(property "Value" "470nF"
 			(at 278.892 232.41 0.0000)
 			(effects
@@
 			)
 		)
-		(property "LCSC" "C1588"
+		(property "LCSC" "C513577"
 			(at 278.13 236.2199 0)
 			(effects
@@
 			)
 		)
-		(property "Value" "1nF"
+		(property "Value" "470nF"
 			(at 379.222 232.41 0.0000)
 			(effects
@@
 			)
 		)
-		(property "LCSC" "C1588"
+		(property "LCSC" "C513577"
 			(at 378.46 236.2199 0)
 			(effects
@@
 			)
 		)
-		(property "Value" "1nF"
+		(property "Value" "470nF"
 			(at 479.552 232.41 0.0000)
 			(effects
@@
 			)
 		)
-		(property "LCSC" "C1588"
+		(property "LCSC" "C513577"
 			(at 478.79 236.2199 0)
 			(effects
