File: boards/core/kicad/amp_b.kicad_sch (KiCad schematic)
At the start: 42 parts, among them J10 SPK B L, J11 SPK B R, U16 TPA3220

Commit message: WIP core banana: schematic, parts, stage-1 ECO, sockets placed
Parts:
- removed J10: SPK B L, aiee:CONN-TH_P5.00_KF301-5.0-2P, symbol aiee:KF301-5.0-2P
- removed J11: SPK B R, aiee:CONN-TH_P5.00_KF301-5.0-2P, symbol aiee:KF301-5.0-2P
- added J24, J26: 24.243 red, aiee:CONN-TH_24.243.1_RED, symbol aiee:24.243.1
- added J25, J27: 24.243 black, aiee:CONN-TH_24.243.2, symbol aiee:24.243.2
Connections:
- net B_SPK_L+: now also J24.1, J24.2
- net B_SPK_L-: now also J25.1, J25.2
- net B_SPK_R+: now also J26.1, J26.2
- net B_SPK_R-: now also J27.1, J27.2
Other:
- moved on the sheet: C301, C302, C304, C306, C307, C308, C309, C310, C311, C312, C316, C317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
