File: boards/core/kicad/linein.kicad_sch (KiCad schematic)
At the start: 28 parts, among them J5 LINE IN, Q6 S8050, U13 ES7243E, U14 TS5A23157, U19 PLR237/T8BK

Commit message: The boards will work on the first spin: independent engineering reviews of Lite and core, fixes and contingencies built…
* First-spin review: the brief each domain reviewer works from

* First-spin review: partial drafts saved before the reviewers' login d…

…ropped

* First-spin review: power, audio, digital and thermal reviews of lite-…

…main and core, with their sims

* core carries its EasyEDA CPL model cache, so its dfm gate runs withou…

…t EasyEDA (red on 403 otherwise); DFM review

* First-spin review: parts pin-to-pad audit of both boards

* Lite board after the first-spin review: amp SDZ, PVDD switch hold-off…

… and soft start, line-in headroom, 5 V loop, RCA slots, HRO USB-C and CH340B, speaker loopback taps; regenerated on hwde c23e27e, all gates pass

Review-2 findings fixed on lite-main as an ECO on the routed board (no
re-route): AUDIO-4/DIGITAL-14, POWER-3/4/10, AUDIO-7, DFM-2, stock swaps.
Also: the speaker loopback taps (task 261029-033806) and the hwde refresh
(task 261029-004401) for this board. Known-unknowns list and its order-step
check (tools/known_unknowns.py). Unit cost at 100: 13.16 (was 13.05).

* core (Plus/Ultra) after the first-spin review: TCA9539 with ESP32 res…

…et, 5 A path via patches and through-hole USB4085, antenna keep-out, PVDD switch SOA and PD-PG gating, OPA1678 headroom, RCA and TOSLINK holes, front IR, 49.152 MHz DAC clock, speaker loopback taps; all gates pass

Review-2 blockers fixed on core: DIGITAL-1/2/PARTS-4, POWER-1, DFM-1, PARTS-7;
THERMAL-1 handled by a lid-pressed heatsink plus firmware governor (no room
for clip holes). Majors: POWER-2/6, AUDIO-1/2/3, DIGITAL-19, DFM-4. Done as an
ECO on the routed board; Ultra zone-B taps left out (no control line).

* First-spin review: every finding's disposition, known-unknowns resolv…

…ed for Lite and Plus (order gate by tier), firmware duties for core, R45 2.2k, honest TPA3221 thermal constraint, Plus/Ultra cost estimate

* Heatsink options for the TPA3221 checked aga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
Parts:
- added C130, C136: 470pF, aiee:C0603, symbol Device:C
- added C131, C137: 1uF, aiee:C0402, symbol Device:C
- added C132: 100nF, aiee:C0402, symbol Device:C
- added Q7: S8050, aiee:SOT-23-3_L3.0-W1.7-P0.95-LS2.9-BR, symbol aiee:S8050_C2146
- added R130, R136: 150k, aiee:R0603, symbol Device:R
- added R131, R135, R137: 10k, aiee:R0402, symbol Device:R
- added R132, R134, R138, R149, R150: 100k, aiee:R0402, symbol Device:R
- added R133: 47k, aiee:R0402, symbol Device:R
- added U20: TS5A23157, aiee:MSOP-10_L3.0-W3.0-P0.50-LS5.0-BL, symbol aiee:TS5A23157DGSR
- C101, C102, C111, C112: value 1uF -> 4.7uF; footprint aiee:C0402 -> aiee:C0603; LCSC C52923 -> C19666
- J5: MPN (none) -> XDJK-0271-1650
Connections:
- net +3V3: now also R132.2, R138.2
- net +5VA: now also C132.1, R135.1, U20.8 (V+)
- net GND: now also C130.2, C132.2, C136.2, Q7.2 (E), R131.2, R134.2, R137.2, R149.2, R150.2, U20.3 (GND)
- net LDIV_L: no longer C101.1
- net LDIV_R: no longer C111.1
- net LSW_L: now also U20.2 (NO1)
- net LSW_R: now also U20.4 (NO2)
- new net ADC_SRC_L: C101.1, U20.10 (COM1)
- new net ADC_SRC_R: C111.1, U20.6 (COM2)
- new net A_SPK_L+: R130.1
- new net A_SPK_R+: R136.1
- new net TAPA_L: C130.1, C131.1, R130.2, R131.1
- new net TAPA_R: C136.1, C137.1, R136.2, R137.1
- new net TAP_B: Q7.1 (B), R133.2, R134.1
- new net TAP_L: C131.2, R132.1, R149.1, U20.9 (NC1)
- new net TAP_R: C137.2, R138.1, R150.1, U20.7 (NC2)
- new net TAP_SEL: Q7.3 (C), R135.2, U20.1 (IN1), U20.5 (IN2)
- new net TAP_SEL_IO: R133.1
Other:
- moved on the sheet: C100, C101, C102, C110, C111, C112, C120, C121, C122, C123, C124, C125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
