File: boards/core/kicad/linein.kicad_sch (KiCad schematic)
At the start: 46 parts, among them J5 LINE IN, Q6 S8050, Q7 S8050, U13 ES7243E, U14 TS5A23157, U19 PLR237/T8BK, U20 TS5A23157

Commit message: core: ESD clamps at the USB-C CC pins and both RCA jacks; speaker and Ethernet lines exempt with reasons (#133)
D6/D9 (NUP2105L) on CC1/CC2, D7/D8 (PESD5V0S2BT) on sub out and line in,
all on B.Cu at their connectors with their own ground vias. KiCad DRC with
schematic parity is clean; check_esd has 0 errors and 4 warnings, judged in
docs/boards/core-esd.md.

Co-Authored-By: Claude Opus 5.5 <noreply@anthropic.com>
Parts:
- added D8: PESD5V0S2BT, aiee:SOT-23_L2.9-W1.3-P1.90-LS2.4-BR, symbol aiee:PESD5V0S2BT,215
Connections:
- net GND: now also D8.3
- net LIN_L: now also D8.1
- net LIN_R: now also D8.2
Other:
- moved on the sheet: C100, C101, C102, C110, C111, C112, C120, C121, C122, C123, C124, C125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
