File: boards/core/kicad/ui.kicad_sch (KiCad schematic)
At the start: 11 parts, among them J3 FFC 20P, SW1 EC11, SW2 BTN1, SW3 BTN2, U18 IRM-H638T

Commit message: The boards will work on the first spin: independent engineering reviews of Lite and core, fixes and contingencies built…
* First-spin review: the brief each domain reviewer works from

* First-spin review: partial drafts saved before the reviewers' login d…

…ropped

* First-spin review: power, audio, digital and thermal reviews of lite-…

…main and core, with their sims

* core carries its EasyEDA CPL model cache, so its dfm gate runs withou…

…t EasyEDA (red on 403 otherwise); DFM review

* First-spin review: parts pin-to-pad audit of both boards

* Lite board after the first-spin review: amp SDZ, PVDD switch hold-off…

… and soft start, line-in headroom, 5 V loop, RCA slots, HRO USB-C and CH340B, speaker loopback taps; regenerated on hwde c23e27e, all gates pass

Review-2 findings fixed on lite-main as an ECO on the routed board (no
re-route): AUDIO-4/DIGITAL-14, POWER-3/4/10, AUDIO-7, DFM-2, stock swaps.
Also: the speaker loopback taps (task 261029-033806) and the hwde refresh
(task 261029-004401) for this board. Known-unknowns list and its order-step
check (tools/known_unknowns.py). Unit cost at 100: 13.16 (was 13.05).

* core (Plus/Ultra) after the first-spin review: TCA9539 with ESP32 res…

…et, 5 A path via patches and through-hole USB4085, antenna keep-out, PVDD switch SOA and PD-PG gating, OPA1678 headroom, RCA and TOSLINK holes, front IR, 49.152 MHz DAC clock, speaker loopback taps; all gates pass

Review-2 blockers fixed on core: DIGITAL-1/2/PARTS-4, POWER-1, DFM-1, PARTS-7;
THERMAL-1 handled by a lid-pressed heatsink plus firmware governor (no room
for clip holes). Majors: POWER-2/6, AUDIO-1/2/3, DIGITAL-19, DFM-4. Done as an
ECO on the routed board; Ultra zone-B taps left out (no control line).

* First-spin review: every finding's disposition, known-unknowns resolv…

…ed for Lite and Plus (order gate by tier), firmware duties for core, R45 2.2k, honest TPA3221 thermal constraint, Plus/Ultra cost estimate

* Heatsink options for the TPA3221 checked aga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
Parts:
- SW2, SW3: MPN (none) -> TS-1187A-B-A-B
- U18: value IRM-H638T -> IRM-3638T; footprint aiee:SENSOR-SMD_IRM-H638T-TR2-TL -> aiee:OPTO-TH_IRM-3638T; symbol aiee:IRM-H638T_TR2 -> aiee:IRM-3638T_C42421366; LCSC C91447 -> C42421366
Connections:
- net GND: no longer U18.1 (GND)
- net IR_IN: now also U18.1 (OUT); no longer U18.3 (VOUT)
- net IR_VCC: now also U18.3 (VCC); no longer U18.4 (VCC)
Other:
- moved on the sheet: C400, R400, R401, R402, R403, SW2, SW3
