File: boards/core/kicad/dac.kicad_sch (KiCad schematic)
At the start: 42 parts, among them J4 SUB OUT, U10 ES9018K2M, U11 OPA1678, U12 PCM5102A, Y1 50MHz

Commit message: The boards will work on the first spin: independent engineering reviews of Lite and core, fixes and contingencies built…
* First-spin review: the brief each domain reviewer works from

* First-spin review: partial drafts saved before the reviewers' login d…

…ropped

* First-spin review: power, audio, digital and thermal reviews of lite-…

…main and core, with their sims

* core carries its EasyEDA CPL model cache, so its dfm gate runs withou…

…t EasyEDA (red on 403 otherwise); DFM review

* First-spin review: parts pin-to-pad audit of both boards

* Lite board after the first-spin review: amp SDZ, PVDD switch hold-off…

… and soft start, line-in headroom, 5 V loop, RCA slots, HRO USB-C and CH340B, speaker loopback taps; regenerated on hwde c23e27e, all gates pass

Review-2 findings fixed on lite-main as an ECO on the routed board (no
re-route): AUDIO-4/DIGITAL-14, POWER-3/4/10, AUDIO-7, DFM-2, stock swaps.
Also: the speaker loopback taps (task 261029-033806) and the hwde refresh
(task 261029-004401) for this board. Known-unknowns list and its order-step
check (tools/known_unknowns.py). Unit cost at 100: 13.16 (was 13.05).

* core (Plus/Ultra) after the first-spin review: TCA9539 with ESP32 res…

…et, 5 A path via patches and through-hole USB4085, antenna keep-out, PVDD switch SOA and PD-PG gating, OPA1678 headroom, RCA and TOSLINK holes, front IR, 49.152 MHz DAC clock, speaker loopback taps; all gates pass

Review-2 blockers fixed on core: DIGITAL-1/2/PARTS-4, POWER-1, DFM-1, PARTS-7;
THERMAL-1 handled by a lid-pressed heatsink plus firmware governor (no room
for clip holes). Majors: POWER-2/6, AUDIO-1/2/3, DIGITAL-19, DFM-4. Done as an
ECO on the routed board; Ultra zone-B taps left out (no control line).

* First-spin review: every finding's disposition, known-unknowns resolv…

…ed for Lite and Plus (order gate by tier), firmware duties for core, R45 2.2k, honest TPA3221 thermal constraint, Plus/Ultra cost estimate

* Heatsink options for the TPA3221 checked aga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
Parts:
- J4: MPN (none) -> XDJK-0271-1650
- R73, R75, R81, R83: value 1.5k -> 1.3k; LCSC C25867 -> C25866
- Y1: value 50MHz -> 49.152MHz; symbol aiee:OT322550MJBA4SL -> aiee:SX3M49.152B10F20TNN; LCSC C717684 -> C7431354
Other:
- moved on the sheet: C142, C57, C58, C59, R71, R72, R73, R74, R75, U11, Y1

Commit message: core: a 2.93 V supervisor (TLV803S) on ESP_EN, so a brownout resets the expander and the PHY clock with the ESP32 (R3-DIGITAL-1); VREF's C64 10 uF -> 100 uF 1206 (R3-AUDIO-1)
U21 sits by R30 and joins ESP_EN and +3V3; C64 moved to the free spot beside
R73 and rejoined to VREF. Prices kept from the committed parts.json; the two
new lines priced live (tools/price_parts.py). DRC clean, zones refilled.
Parts:
- C64: value 10uF -> 100uF; footprint aiee:C0603 -> aiee:C1206; LCSC C19702 -> C15008
Changed lines of the file:
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@@
 			)
 		)
-		(property "Value" "10uF"
+		(property "Value" "100uF"
 			(at 238.252 99.06 0.0000)
 			(effects
@@
 			)
 		)
-		(property "Footprint" "aiee:C0603"
+		(property "Footprint" "aiee:C1206"
 			(at 235.9152 93.98 0.0000)
 			(effects
@@
 			)
 		)
-		(property "LCSC" "C19702"
+		(property "LCSC" "C15008"
 			(at 237.49 102.8699 0)
 			(effects
