File: boards/core/kicad/dac.kicad_sch (KiCad schematic)
At the start: 42 parts, among them J4 SUB OUT, U10 ES9018K2M, U11 OPA1678, U12 PCM5102A, Y1 49.152MHz

Commit message: core: ESD clamps at the USB-C CC pins and both RCA jacks; speaker and Ethernet lines exempt with reasons (#133)
D6/D9 (NUP2105L) on CC1/CC2, D7/D8 (PESD5V0S2BT) on sub out and line in,
all on B.Cu at their connectors with their own ground vias. KiCad DRC with
schematic parity is clean; check_esd has 0 errors and 4 warnings, judged in
docs/boards/core-esd.md.

Co-Authored-By: Claude Opus 5.5 <noreply@anthropic.com>
Parts:
- added D7: PESD5V0S2BT, aiee:SOT-23_L2.9-W1.3-P1.90-LS2.4-BR, symbol aiee:PESD5V0S2BT,215
Connections:
- net GND: now also D7.3
- net SUB1_OUT: now also D7.1
- net SUB2_OUT: now also D7.2
Changed lines of the file:
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@@
 		)
 		(property "Value" "SUB OUT"
-			(at 504.7246 92.71 0.0000)
+			(at 494.5646 92.71 0.0000)
 			(effects
 				(font
@@
 		)
 	)
+	(symbol
+		(lib_id "aiee:PESD5V0S2BT,215")
+		(at 528.32 104.14 0)
+		(unit 1)
+		(exclude_from_sim no)
+		(in_bom yes)
+		(on_board yes)
+		(dnp no)
+		(fields_autoplaced no)
+		(property "Reference" "D7"
+			(at 527.3306 115.57 0.0000)
+			(effects
+				(font
+					(size 1.27 1.27)
+				)
+				(justify left)
+			)
+		)
+		(property "Value" "PESD5V0S2BT"
+			(at 516.89 92.71 0.0000)
+			(effects
+				(font
+					(size 1.27 1.27)
+				)
+				(justify right)
+			)
+		)
+		(property "Footprint" "aiee:SOT-23_L2.9-W1.3-P1.90-LS2.4-BR"
+			(at 528.32 86.36 0.0000)
+			(effects
+				(font
+					(size 1.27 1.27)
+				)
+				(hide yes)
+			)
+		)
+		(property "LCSC" "C49338"
+			(at 530.86 109.2199 0)
+			(effects
+				(font
+					(size 1.27 1.27)
+				)
+				(justify left)
+			)
+		)
+		(property "MPN" "PESD5V0S2BT,215"
+			(at 530.86 109.2199 0)
+			(effects
+				(font
+					(size 1.27 1.27)
+				)
+				(justify left)
+			)
+		)
+		(pin "1"
+		)
+		(pin "2"
+		)
+		(pin "3"
+		)
+		(instances
+			(project "dac"
+				(path "/caa78795-1512-4865-b6c8-dd81dc66e7f0"
+					(reference "D7")
+					(unit 1)
+				)
+			)
+		)
+	)
+	(symbol
+		(lib_id "power:GND")
+		(at 528.32 91.44 0)
+		(unit 1)
+		(exclude_from_sim no)
+		(in_bom yes)
+		(on_board yes)
+		(dnp no)
+		(fields_autoplaced no)
+		(property "Reference" "#PWR5060"
+			(at 528.32 85.09 0.0000)
+			(effects
+				(font
+					(size 1.27 1.27)
+				)
+				(justify left)
+				(hide yes)
+			)
+		)
+		(property "Value" "GND"
+			(at 529.59 95.25 0.0000)
+			(effects
+				(font
+					(size 1.27 1.27)
+				)
+				(justify left)
+			)
+		)
+		(pin "1"
+		)
+		(instances
+			(project "dac"
+				(path "/caa78795-1512-4865-b6c8-dd81dc66e7f0"
+					(reference "#PWR5060")
+					(unit 1)
+				)
+			)
+		)
+	)
 	(wire
 		(pts
@@
 		(pts
 			(xy 505.46 104.14) (xy 505.46 106.68)
+		)
+		(stroke
+			(width 0)
+			(type default)
+		)
+	)
+	(wire
+		(pts
+			(xy 523.24 114.3) (xy 523.24 116.84)
+		)
+		(stroke
+			(width 0)
+			(type default)
+		)
+	)
+	(wire
+		(pts
+			(xy 533.4 114.3) (xy 533.4 116.84)
+		)
+		(stroke
+			(width 0)
+			(type default)
+		)
+	)
+	(wire
+		(pts
+			(xy 528.32 93.98) (xy 528.32 91.44)
 		)
 		(stroke
@@
 		)
 	)
+	(label "SUB1_OUT"
+		(at 523.24 116.84 270)
+		(effects
+			(font
+				(size 1.27 1.27)
+			)
+			(justify right bottom)
+		)
+	)
+	(label "SUB2_OUT"
+		(at 533.4 116.84 270)
+		(effects
+			(font
+				(size 1.27 1.27)
+			)
+			(justify right bottom)
+		)
+	)
+	(label "GND"
+		(at 528.32 91.44 90)
+		(effects
+			(font
+				(size 1.27 1.27)
+			)
+			(justify left bottom)
+		)
+	)
