File: boards/core/kicad/amp_a.kicad_sch (KiCad schematic)
At the start: 44 parts, among them J6 SPK A L, J7 SPK A R, U15 TPA3221

Commit message: The boards will work on the first spin: independent engineering reviews of Lite and core, fixes and contingencies built…
* First-spin review: the brief each domain reviewer works from

* First-spin review: partial drafts saved before the reviewers' login d…

…ropped

* First-spin review: power, audio, digital and thermal reviews of lite-…

…main and core, with their sims

* core carries its EasyEDA CPL model cache, so its dfm gate runs withou…

…t EasyEDA (red on 403 otherwise); DFM review

* First-spin review: parts pin-to-pad audit of both boards

* Lite board after the first-spin review: amp SDZ, PVDD switch hold-off…

… and soft start, line-in headroom, 5 V loop, RCA slots, HRO USB-C and CH340B, speaker loopback taps; regenerated on hwde c23e27e, all gates pass

Review-2 findings fixed on lite-main as an ECO on the routed board (no
re-route): AUDIO-4/DIGITAL-14, POWER-3/4/10, AUDIO-7, DFM-2, stock swaps.
Also: the speaker loopback taps (task 261029-033806) and the hwde refresh
(task 261029-004401) for this board. Known-unknowns list and its order-step
check (tools/known_unknowns.py). Unit cost at 100: 13.16 (was 13.05).

* core (Plus/Ultra) after the first-spin review: TCA9539 with ESP32 res…

…et, 5 A path via patches and through-hole USB4085, antenna keep-out, PVDD switch SOA and PD-PG gating, OPA1678 headroom, RCA and TOSLINK holes, front IR, 49.152 MHz DAC clock, speaker loopback taps; all gates pass

Review-2 blockers fixed on core: DIGITAL-1/2/PARTS-4, POWER-1, DFM-1, PARTS-7;
THERMAL-1 handled by a lid-pressed heatsink plus firmware governor (no room
for clip holes). Majors: POWER-2/6, AUDIO-1/2/3, DIGITAL-19, DFM-4. Done as an
ECO on the routed board; Ultra zone-B taps left out (no control line).

* First-spin review: every finding's disposition, known-unknowns resolv…

…ed for Lite and Plus (order gate by tier), firmware duties for core, R45 2.2k, honest TPA3221 thermal constraint, Plus/Ultra cost estimate

* Heatsink options for the TPA3221 checked aga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
Parts:
- J6, J7: MPN (none) -> KF301-5.0-2P

Commit message: TPA3221 heatsink the person doesn't have to fit: a JLC-fittable board-mount part or a pad-down amp
* First-spin review: the brief each domain reviewer works from

* First-spin review: partial drafts saved before the reviewers' login d…

…ropped

* First-spin review: power, audio, digital and thermal reviews of lite-…

…main and core, with their sims

* core carries its EasyEDA CPL model cache, so its dfm gate runs withou…

…t EasyEDA (red on 403 otherwise); DFM review

* First-spin review: parts pin-to-pad audit of both boards

* Lite board after the first-spin review: amp SDZ, PVDD switch hold-off…

… and soft start, line-in headroom, 5 V loop, RCA slots, HRO USB-C and CH340B, speaker loopback taps; regenerated on hwde c23e27e, all gates pass

Review-2 findings fixed on lite-main as an ECO on the routed board (no
re-route): AUDIO-4/DIGITAL-14, POWER-3/4/10, AUDIO-7, DFM-2, stock swaps.
Also: the speaker loopback taps (task 261029-033806) and the hwde refresh
(task 261029-004401) for this board. Known-unknowns list and its order-step
check (tools/known_unknowns.py). Unit cost at 100: 13.16 (was 13.05).

* core (Plus/Ultra) after the first-spin review: TCA9539 with ESP32 res…

…et, 5 A path via patches and through-hole USB4085, antenna keep-out, PVDD switch SOA and PD-PG gating, OPA1678 headroom, RCA and TOSLINK holes, front IR, 49.152 MHz DAC clock, speaker loopback taps; all gates pass

Review-2 blockers fixed on core: DIGITAL-1/2/PARTS-4, POWER-1, DFM-1, PARTS-7;
THERMAL-1 handled by a lid-pressed heatsink plus firmware governor (no room
for clip holes). Majors: POWER-2/6, AUDIO-1/2/3, DIGITAL-19, DFM-4. Done as an
ECO on the routed board; Ultra zone-B taps left out (no control line).

* First-spin review: every finding's disposition, known-unknowns resolv…

…ed for Lite and Plus (order gate by tier), firmware duties for core, R45 2.2k, honest TPA3221 thermal constraint, Plus/Ultra cost estimate

* Heatsink options for the TPA3221 checked against the lead's order;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
Parts:
- U15: value TPA3221 -> TPA3220; footprint aiee:HTSSOP-44_L14.0-W6.1-P0.64-LS8.1-BL -> aiee:HTSSOP-44-1EP_L14.0-W6.1-P0.64-LS8.1-EP7.3x4.43; symbol aiee:TPA3221DDVR -> aiee:TPA3220DDWR; LCSC C475500 -> C2879306
Connections:
- net GND: now also U15.45 (GND)
Other:
- moved on the sheet: C226, C228, C229, C231, C232, C234, C235, C237, J6, J7, L1, L2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

Commit message: core amp-area ECO (#121): TPA3220 PVDD HF pairs under the pins and BST caps at the row ends (R3-AMP-1/2), U15's input caps at the IN pins (R3-LAYOUT-1); two-sided build, every gate passes
Parts:
- C207, C209: footprint aiee:C0805 -> aiee:C1206; LCSC C28323 -> C282823
Changed lines of the file:
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@@
 			)
 		)
-		(property "Footprint" "aiee:C0805"
+		(property "Footprint" "aiee:C1206"
 			(at 251.1552 35.56 0.0000)
 			(effects
@@
 			)
 		)
-		(property "LCSC" "C28323"
+		(property "LCSC" "C282823"
 			(at 252.73 44.4499 0)
 			(effects
@@
 			)
 		)
-		(property "Footprint" "aiee:C0805"
+		(property "Footprint" "aiee:C1206"
 			(at 286.7152 35.56 0.0000)
 			(effects
@@
 			)
 		)
-		(property "LCSC" "C28323"
+		(property "LCSC" "C282823"
 			(at 288.29 44.4499 0)
 			(effects
