File: boards/core/kicad/amp_a.kicad_sch (KiCad schematic)
At the start: 44 parts, among them J6 SPK A L, J7 SPK A R, U15 TPA3220

Commit message: Revert "core amp-area layout ECO: TPA3220 bootstrap and PVDD HF caps at their pins, input caps at the IN pins"
This reverts commit f0eb13530c5fd08d8df6501fd36629fa8401f02f.
Parts:
- C207, C209: footprint aiee:C1206 -> aiee:C0805; LCSC C282823 -> C28323
Changed lines of the file:
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@@
 			)
 		)
-		(property "Footprint" "aiee:C1206"
+		(property "Footprint" "aiee:C0805"
 			(at 251.1552 35.56 0.0000)
 			(effects
@@
 			)
 		)
-		(property "LCSC" "C282823"
+		(property "LCSC" "C28323"
 			(at 252.73 44.4499 0)
 			(effects
@@
 			)
 		)
-		(property "Footprint" "aiee:C1206"
+		(property "Footprint" "aiee:C0805"
 			(at 286.7152 35.56 0.0000)
 			(effects
@@
 			)
 		)
-		(property "LCSC" "C282823"
+		(property "LCSC" "C28323"
 			(at 288.29 44.4499 0)
 			(effects
