File: boards/core/kicad/amp_a.kicad_sch (KiCad schematic)
At the start: 44 parts, among them J6 SPK A L, J7 SPK A R, U15 TPA3220

Commit message: core's class-D outputs are damped with no speaker: the 4.7R snubbers get 470nF Zobel caps (#137)
The 8 per-leg snubber caps C228/C231/C234/C237/C326/C329/C332/C335 go from
1nF to 470nF/50V X7R 0603 (Yageo CC0603KRX7R9BB474, LCSC C513577). Same
footprints: board_update changed only value and LCSC fields, no copper.
Open-load peak +39.7 dB -> +15.8 dB (ngspice, docs/boards/sims/zobel_sweep.py);
4/6/8 ohm responses move under 0.6 dB. Test tones refuse a sine above 5 kHz
louder than -16 dBFS without force, so the 0603 resistors stay in rating.
Lite checked the same way and left as it is (docs/boards/core-zobel.md).

Co-Authored-By: Claude Opus 5.5 <noreply@anthropic.com>
Parts:
- C228, C231, C234, C237: value 1nF -> 470nF; LCSC C1588 -> C513577
Changed lines of the file:
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@@
 			)
 		)
-		(property "Value" "1nF"
+		(property "Value" "470nF"
 			(at 155.702 119.38 0.0000)
 			(effects
@@
 			)
 		)
-		(property "LCSC" "C1588"
+		(property "LCSC" "C513577"
 			(at 154.94 123.1899 0)
 			(effects
@@
 			)
 		)
-		(property "Value" "1nF"
+		(property "Value" "470nF"
 			(at 256.032 119.38 0.0000)
 			(effects
@@
 			)
 		)
-		(property "LCSC" "C1588"
+		(property "LCSC" "C513577"
 			(at 255.27 123.1899 0)
 			(effects
@@
 			)
 		)
-		(property "Value" "1nF"
+		(property "Value" "470nF"
 			(at 356.362 119.38 0.0000)
 			(effects
@@
 			)
 		)
-		(property "LCSC" "C1588"
+		(property "LCSC" "C513577"
 			(at 355.6 123.1899 0)
 			(effects
@@
 			)
 		)
-		(property "Value" "1nF"
+		(property "Value" "470nF"
 			(at 456.692 119.38 0.0000)
 			(effects
@@
 			)
 		)
-		(property "LCSC" "C1588"
+		(property "LCSC" "C513577"
 			(at 455.93 123.1899 0)
 			(effects
