File: boards/core/kicad/power_in.kicad_sch (KiCad schematic)
At the start: 36 parts, among them J1 USB4085-GF-A, Q1 AO4485, Q2 2N7002, Q3 MMDT3904, U1 CH224Q, U2 USBLC6-2SC6, U3 INA186A1

Commit message: WIP core banana: speaker pours as one staircase polygon per net, In2 pin links, C4/C8 (R5-PA-1), DAL-7, stubs ripped
Parts:
- C4: value 100nF -> 220nF; LCSC C14663 -> C344195
- C8: value 2.2uF -> 4.7uF; LCSC C377773 -> C1779
Changed lines of the file:
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@@
 			)
 		)
-		(property "Value" "100nF"
+		(property "Value" "220nF"
 			(at 315.468 93.98 0.0000)
 			(effects
@@
 			)
 		)
-		(property "LCSC" "C14663"
+		(property "LCSC" "C344195"
 			(at 321.31 97.7899 0)
 			(effects
@@
 			)
 		)
-		(property "Value" "2.2uF"
+		(property "Value" "4.7uF"
 			(at 339.852 93.98 0.0000)
 			(effects
@@
 			)
 		)
-		(property "LCSC" "C377773"
+		(property "LCSC" "C1779"
 			(at 339.09 97.7899 0)
 			(effects
