File: boards/lite-main/kicad/lite-main.kicad_sch (KiCad schematic)
At the start: 134 parts, among them J1 USB4105-GF-A-120, J2 RCA line in, J3 RCA sub out, J4 DB128V-5.08-4P, Q1 AO4485, Q2 MMBT3904, Q3 MMBT3904, Q4 MMBT3904, SW1 TS-1187A, SW2 TS-1187A, SW3 TS-1187A, U1 CH224A, U2 TPS54302, U3 SY8089A1AAC, U4 LP5907-3.3, U5 ESP32-WROVER-E-N8R8, U6 CH340C, U7 ES8388, U8 TPA3118D2, U9 IRM-3638T

Commit message: The boards will work on the first spin: independent engineering reviews of Lite and core, fixes and contingencies built…
* First-spin review: the brief each domain reviewer works from

* First-spin review: partial drafts saved before the reviewers' login d…

…ropped

* First-spin review: power, audio, digital and thermal reviews of lite-…

…main and core, with their sims

* core carries its EasyEDA CPL model cache, so its dfm gate runs withou…

…t EasyEDA (red on 403 otherwise); DFM review

* First-spin review: parts pin-to-pad audit of both boards

* Lite board after the first-spin review: amp SDZ, PVDD switch hold-off…

… and soft start, line-in headroom, 5 V loop, RCA slots, HRO USB-C and CH340B, speaker loopback taps; regenerated on hwde c23e27e, all gates pass

Review-2 findings fixed on lite-main as an ECO on the routed board (no
re-route): AUDIO-4/DIGITAL-14, POWER-3/4/10, AUDIO-7, DFM-2, stock swaps.
Also: the speaker loopback taps (task 261029-033806) and the hwde refresh
(task 261029-004401) for this board. Known-unknowns list and its order-step
check (tools/known_unknowns.py). Unit cost at 100: 13.16 (was 13.05).

* core (Plus/Ultra) after the first-spin review: TCA9539 with ESP32 res…

…et, 5 A path via patches and through-hole USB4085, antenna keep-out, PVDD switch SOA and PD-PG gating, OPA1678 headroom, RCA and TOSLINK holes, front IR, 49.152 MHz DAC clock, speaker loopback taps; all gates pass

Review-2 blockers fixed on core: DIGITAL-1/2/PARTS-4, POWER-1, DFM-1, PARTS-7;
THERMAL-1 handled by a lid-pressed heatsink plus firmware governor (no room
for clip holes). Majors: POWER-2/6, AUDIO-1/2/3, DIGITAL-19, DFM-4. Done as an
ECO on the routed board; Ultra zone-B taps left out (no control line).

* First-spin review: every finding's disposition, known-unknowns resolv…

…ed for Lite and Plus (order gate by tier), firmware duties for core, R45 2.2k, honest TPA3221 thermal constraint, Plus/Ultra cost estimate

* Heatsink options for the TPA3221 checked aga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
Parts:
- added C19: 4.7uF, Capacitor_SMD:C_0603_1608Metric, symbol Device:C
- added C25: 22uF, Capacitor_SMD:C_0805_2012Metric, symbol Device:C
- added C26: 47nF, Capacitor_SMD:C_0603_1608Metric, symbol Device:C
- added C81, C83: 470pF, Capacitor_SMD:C_0603_1608Metric, symbol Device:C
- added C82, C84: 1uF, Capacitor_SMD:C_0603_1608Metric, symbol Device:C
- added R66, R68: 100k, Resistor_SMD:R_0603_1608Metric, symbol Device:R
- added R67, R69: 10k, Resistor_SMD:R_0603_1608Metric, symbol Device:R
- C9: value 100pF -> 47pF; LCSC C14858 -> C1671
- J1: value USB4105-GF-A-120 -> TYPE-C-31-M-12; footprint aiee:USB-C-SMD_MC-311D -> aiee:USB-C_SMD-TYPE-C-31-M-12_1; symbol aiee:USB4105-GF-A-120 -> aiee:TYPE-C-31-M-12; LCSC C5184243 -> C165948
- R30, R33: value 10k -> 15k; LCSC C25804 -> C22809
- R54: value 100k -> 10k; LCSC C25803 -> C25804
- R6: value 47k -> 220k; LCSC C25819 -> C22961
- U6: value CH340C -> CH340B; symbol aiee:CH340C -> aiee:CH340B; LCSC C84681 -> C81010
Connections:
- net +5V: now also C25.1
- net AMP_SDZ: now also C26.1
- net GND: now also J1.A1B12 (GND), J1.B1A12 (GND), C25.2, C26.2, C81.2, C83.2, R67.2, R69.2; no longer J1.A1-B12 (GND), J1.B1-A12 (GND)
- net PSW_G: now also C19.2
- net SPK_L_P: now also R66.1
- net SPK_R_P: now also R68.1
- net VBUS: now also J1.A4B9 (VBUS), J1.B4A9 (VBUS), C19.1; no longer J1.A4-B9 (VBUS), J1.B4-A9 (VBUS)
- net TAP_R_C: now reaches U7.21 (RIN2)
- net TAP_R_C: now also C84.2
- net TAP_L_C: now reaches U7.22 (LIN2)
- net TAP_L_C: now also C82.2
- new net TAP_L: C81.1, C82.1, R66.2, R67.1
- new net TAP_R: C83.1, C84.1, R68.2, R69.1
- no-connect marks 31 -> 29
Other:
- moved on the sheet: C1, C10, C11, C12, C13, C14, C15, C16, C17, C18, C2, C20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

Commit message: Lite's VBUS TVS is an SMBJ22A: its 22 V standoff covers a 20 V PD contract's 21 V, and Lite passes hwde 4827325
D1 SMBJ20A (C364296, 20 V standoff) -> SMBJ22A (MDD C113993, same SMB
footprint and pinout), as a same-footprint swap on the routed board
(board_update; copper and drill unchanged). Schematic, netlist, parts,
BOM/CPL, prebuy and gates regenerated; known-unknowns power:10 and
thermal:30 resolved.
Parts:
- D1: value SMBJ20A -> SMBJ22A; symbol aiee:SMBJ20A_C364296 -> aiee:SMBJ22A_C113993; LCSC C364296 -> C113993
Changed lines of the file:
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@@
 	)
 	(symbol
-		(lib_id "aiee:SMBJ20A_C364296")
+		(lib_id "aiee:SMBJ22A_C113993")
 		(at 320.04 90.17 0)
 		(unit 1)
@@
 			)
 		)
-		(property "Value" "SMBJ20A"
+		(property "Value" "SMBJ22A"
 			(at 316.7646 93.47 0.0000)
 			(effects
@@
 			)
 		)
-		(property "LCSC" "C364296"
+		(property "LCSC" "C113993"
 			(at 322.58 95.2499 0)
 			(effects
