File: boards/lite-main/kicad/lite-main.kicad_sch (KiCad schematic)
At the start: 148 parts, among them J1 TYPE-C-31-M-12, J2 RCA line in, J3 RCA sub out, J4 24.243 red, J5 24.243 black, J6 24.243 red, J7 24.243 black, Q1 AO4485, Q2 MMBT3904, Q3 MMBT3904, Q4 MMBT3904, SW1 TS-1187A, SW2 TS-1187A, SW3 TS-1187A, U1 CH224A, U2 TPS54302, U3 SY8089A1AAC, U4 LP5907-3.3, U5 ESP32-WROVER-E-N8R8, U6 CH340B, U7 ES8388, U8 TPA3118D2, U9 IRM-3638T

Commit message: Lite and core converge: review rounds against app notes, reference designs and known field issues until a round finds n…
* Review round 2: the brief each reviewer works from (app notes, refere…

…nce designs, field issues)

* Review round 2: partial drafts (power, amp, audio, system, layout) an…

…d their tests, saved before the session dropped

* Review round 2: amp review (2 majors on core: bootstrap and PVDD HF c…

…ap placement) and its tests

* Review round 2: audio-chain review (3 majors: core VREF filtering, Li…

…te sub-out power-loss thump, core DJ-direct subs silent) and its sims

* Review round 2: power review (4 majors: core PVDD turn-on SOA regress…

…ion, charger peak current under the average governor, core VBUS unknown, EPR step) and its benches

* Review round 2: digital review (3 majors: core GPIO0 strap on interna…

…l resets, LAN8720 PHY address, Ultra front board undriven) and its tests

* Review round 2: system/field review (4 majors: governor and clipping,…

… Lite L1 thermal, core GPIO0 on restart, DJ-direct thermal on core) and its tests

* Firmware after review round 2: the governor limits on the unclipped p…

…rogram and each block's peak, Lite's L1 thermal limit, core reads the charger's PDOs and waits for EPR, 500 ms PVDD soft start, PHY clock off before a restart, OTW step-down, amps held across an input change and until the codec settles, input kept in NVS

R3-SYSTEM-1/2/3/5, R3-POWER-2(firmware half)/3/4/5, R3-DIGITAL-1(firmware half); round-1 duties L1 L4 C1 C2 C5. Host tests pass (make in firmware/test).

* Merge branch 'main' of /hive/run/main.bundle into hive/w-261030-15165…

…6-0a0fabd0ce

* Review round 2: layout/DFM/thermal review (blocker: core J4/J5 RCA fo…

…otprints never took round 1's leg holes; major: core amp input routing) and its tests

* Lite's sub outs mute on power loss (review-3 R3-AUDIO-2): a +5V sense…

… holds two back-to-back 2N7002s off; when +5V drops they short SUB_L/SUB_R to GND from a 22 uF reservoir for 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
Parts:
- added C90: 22uF, Capacitor_SMD:C_0805_2012Metric, symbol Device:C
- added Q11, Q12: MMBT3904, aiee:SOT-23-3_L2.9-W1.3-P1.90-LS2.4-BR, symbol aiee:MMBT3904-C20526
- added Q13, Q14, Q15: 2N7002, aiee:SOT-23-3_L2.9-W1.3-P1.90-LS2.4-BR, symbol aiee:2N7002
- added R80: 120k, Resistor_SMD:R_0603_1608Metric, symbol Device:R
- added R81: 22k, Resistor_SMD:R_0603_1608Metric, symbol Device:R
- added R82: 47k, Resistor_SMD:R_0603_1608Metric, symbol Device:R
- R36, R38: value 100R -> 1k; LCSC C22775 -> C21190
Connections:
- net +5V: now also Q11.1 (B), Q11.3 (C), R80.1
- net GND: now also C90.2, Q12.2 (E), Q14.3 (D), R81.2
- net SUB_L: now also Q13.3 (D)
- net SUB_R: now also Q15.3 (D)
- new net MUTE_DET: Q12.1 (B), R80.2, R81.1
- new net MUTE_RES: C90.1, Q11.2 (E), R82.1
- new net MUTE_S: Q13.2 (S), Q14.2 (S), Q15.2 (S)
- new net SUB_MUTE: Q12.3 (C), Q13.1 (G), Q14.1 (G), Q15.1 (G), R82.2
