File: boards/lite-main/kicad/lite-main.kicad_sch (KiCad schematic)
At the start: 157 parts, among them J1 TYPE-C-31-M-12, J2 RCA line in, J3 RCA sub out, J4 24.243 red, J5 24.243 black, J6 24.243 red, J7 24.243 black, Q1 AO4485, Q11 MMBT3904, Q12 MMBT3904, Q13 2N7002, Q14 2N7002, Q15 2N7002, Q2 MMBT3904, Q3 MMBT3904, Q4 MMBT3904, SW1 TS-1187A, SW2 TS-1187A, SW3 TS-1187A, U1 CH224A, U2 TPS54302, U3 SY8089A1AAC, U4 LP5907-3.3, U5 ESP32-WROVER-E-N8R8, U6 CH340B, U7 ES8388, U8 TPA3118D2, U9 IRM-3638T

Commit message: lite-main: ESD clamps at the USB-C, line-in and sub-out; speaker posts exempt with reasons (#133)
D3/D4 NUP2105L on CC2/CC1, U10 USBLC6-2SC6 on D+/D-, D5/D6 PESD5V0S2BT on
the two RCA jacks, all on B.Cu by their connectors (kicad/gen/esd_eco.py).
The USB pair's first 2-3 mm under J1 is redone so CC2 and the clamps can
reach the pins. Fab regenerated; DRC with parity clean; dfm passes with
bottom-side waivers.

Co-Authored-By: Claude Opus 5.5 <noreply@anthropic.com>
Parts:
- added D3, D4: NUP2105L, aiee:SOT-23-3_L2.9-W1.3-P1.90-LS2.4-BL-2, symbol aiee:NUP2105LT1G
- added D5, D6: PESD5V0S2BT, aiee:SOT-23_L2.9-W1.3-P1.90-LS2.4-BR, symbol aiee:PESD5V0S2BT,215
- added U10: USBLC6-2SC6, aiee:SOT-23-6_L2.9-W1.6-P0.95-LS2.8-BL, symbol aiee:USBLC6-2SC6_C2687116
Connections:
- net CC1: now also D4.1
- net CC2: now also D3.1
- net GND: now also D3.3, D4.3, D5.3, D6.3, U10.2 (GND)
- net LINEIN_L: now also D5.1
- net LINEIN_R: now also D5.2
- net SUB_L: now also D6.1
- net SUB_R: now also D6.2
- net USB_DM: now also U10.4 (I/O2)
- net USB_DP: now also U10.6 (I/O1)
- no-connect marks 29 -> 34
Other:
- moved on the sheet: C1, C10, C11, C12, C13, C14, C15, C16, C17, C18, C19, C2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

Commit message: lite-main ESD: top-side only (the person: Lite stays cheap); L1-L4 attr fix
Replaces the bottom-side clamps. Six PESDNC2FD5VB (C110694, DFN1006) on F.Cu:
D3/D4 at line-in J2, D5/D6 at sub-out J3, D7/D8 on USB D+/D- left of J1.
CC1/CC2 exempt: no top-side spot ahead of the CH224A, 2 mm from J1.
L1-L4 XR0850 (attr through_hole -> smd) via fpfix, board and lib, so
bom-cpl keeps them on the SMT line (hive-hwde #415 check_fp_attr).
check_esd 0 errors / 2 warnings (USB_DM: 2 vias, 13.8 mm); DRC with parity
0/0/0; fab regenerated with no Bottom CPL rows; hwcheck test passes.

Co-Authored-By: Claude Opus 5.5 <noreply@anthropic.com>
Parts:
- removed U10: USBLC6-2SC6, aiee:SOT-23-6_L2.9-W1.6-P0.95-LS2.8-BL, symbol aiee:USBLC6-2SC6_C2687116
- added D7, D8: PESDNC2FD5VB, aiee:DFN1006-2L-BI, symbol aiee:PESDNC2FD5VB
- D3, D4: value NUP2105L -> PESDNC2FD5VB; footprint aiee:SOT-23-3_L2.9-W1.3-P1.90-LS2.4-BL-2 -> aiee:DFN1006-2L-BI; symbol aiee:NUP2105LT1G -> aiee:PESDNC2FD5VB; LCSC C14486 -> C110694
- D5, D6: value PESD5V0S2BT -> PESDNC2FD5VB; footprint aiee:SOT-23_L2.9-W1.3-P1.90-LS2.4-BR -> aiee:DFN1006-2L-BI; symbol aiee:PESD5V0S2BT,215 -> aiee:PESDNC2FD5VB; LCSC C49338 -> C110694
Connections:
- net CC1: no longer D4.1
- net CC2: no longer D3.1
- net GND: now also D3.2, D4.2, D5.2, D6.2, D7.2, D8.2; no longer D3.3, D4.3, D5.3, D6.3
- net LINEIN_L: now also D3.1; no longer D5.1
- net LINEIN_R: now also D4.1; no longer D5.2
- net SUB_L: now also D5.1; no longer D6.1
- net SUB_R: now also D6.1; no longer D6.2
- net USB_DM: now also D8.1
- net USB_DP: now also D7.1
- no-connect marks 34 -> 29
Other:
- moved on the sheet: C1, C10, C11, C12, C13, C14, C15, C16, C17, C18, C19, C2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
