File: boards/lite-main/kicad/lite-main.kicad_pcb (KiCad board)
At the start: 2 copper layers, 118 x 90 mm, 167 parts, among them J1 TYPE-C-31-M-12, J2 RCA line in, J3 RCA sub out, J4 24.243 red, J5 24.243 black, J6 24.243 red, J7 24.243 black, Q1 AO4485, Q11 MMBT3904, Q12 MMBT3904, Q13 2N7002, Q14 2N7002, Q15 2N7002, Q2 MMBT3904, Q3 MMBT3904, Q4 MMBT3904, SW1 TS-1187A, SW2 TS-1187A, SW3 TS-1187A, U1 CH224A, U2 TPS54302, U3 SY8089A1AAC, U4 LP5907-3.3, U5 ESP32-WROVER-E-N8R8, U6 CH340B, U7 ES8388, U8 TPA3118D2, U9 IRM-3638T

Commit message: lite-main pre-order round: vias off pads, I2S respaced, VBUS stubs, box hole axis
check_wicking 15 -> 0; I2S crosstalk now inside the noise margin; VBUS out of J1
widened; banana holes use the part's x in every box (R6-M2); the stale
architecture/constraints.json is gone. See docs/boards/lite-preorder.md.

Co-Authored-By: Claude Opus 5.5 <noreply@anthropic.com>
Routing:
- net GND: track 166.9 -> 177.0 mm, vias 128 -> 129
- net /MUTE_S: track 7.52 -> 11.0 mm
- net /PSW_G: track 27.3 -> 29.1 mm
- net +5V: track 87.2 -> 85.5 mm, vias 6 -> 4
- net VBUS: track 100.5 -> 102.1 mm
- net /SUB_L: track 19.0 -> 20.5 mm
- net /MUTE_DET: track 28.2 -> 29.6 mm
- net /TAP_R_C: track 8.98 -> 9.61 mm

Commit message: lite-main: keep the second +5V vias at L5 and C25, off the pads
check_current needs 2 vias at both layer changes (0.8 A).

Co-Authored-By: Claude Opus 5.5 <noreply@anthropic.com>
Routing:
- net +5V: track 85.5 -> 88.9 mm, vias 4 -> 6
Changed lines of the file:
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@@
+	)
+	(segment
+		(start 86.3 100.85)
+		(end 86.6 100.3)
+		(width 0.405)
+		(layer "F.Cu")
+		(net "+5V")
 	)
 	(segment
@@
 	)
 	(segment
+		(start 84.5 94)
+		(end 84.3 93.2)
+		(width 0.405)
+		(layer "F.Cu")
+		(net "+5V")
+	)
+	(segment
 		(start 73.5 89.45)
 		(end 73.5 89.55)
@@
 	)
 	(via
+		(at 86.3 100.85)
+		(size 0.6)
+		(drill 0.3)
+		(layers "F.Cu" "B.Cu")
+		(net "+5V")
+	)
+	(via
+		(at 84.5 94)
+		(size 0.6)
+		(drill 0.3)
+		(layers "F.Cu" "B.Cu")
+		(net "+5V")
+	)
+	(via
 		(at 69.9 87.25)
 		(size 0.6)
@@
 		(width 0.405)
 		(layer "B.Cu")
+		(net "+5V")
+	)
+	(segment
+		(start 85.9 98.95)
+		(end 86.3 100.85)
+		(width 0.405)
+		(layer "B.Cu")
