File: boards/ultra-front/kicad/ultra-front.kicad_pcb (KiCad board)
At the start: 2 copper layers, 110 x 40 mm, 40 parts, among them J1 FPC-05F-20PH20, J2 FPC-05FB-12PH20, Q1 AO3400A, SW1 TS-1187A-B-A-B, SW2 TS-1187A-B-A-B, SW3 TS-1187A-B-A-B, SW4 EC11E1834403, U1 TCA9535PWR, U2 IRM-H638T/TR2

Commit message: ultra-front: ESD clamps at the switches (R5-UF-2)
D2/D3 PESD5V0S2BT (C49338, as on core): D2 on BTN2/BTN1 between SW1 and
SW2, D3 on BTN3/ENC_SW between SW2 and SW3, each GND pin on its own via.
Schematic generator, parts, PCB (board_update + kicad/gen/esd_eco.py), fab
regenerated, README, bom-estimate and product.md totals updated.
docs/boards/ultra-front-esd.md has the layout reasoning.

Co-Authored-By: Claude Opus 5.5 <noreply@anthropic.com>
Parts:
- added D2: PESD5V0S2BT, aiee:SOT-23_L2.9-W1.3-P1.90-LS2.4-BR, F.Cu at (74.0, 40.8)
- added D3: PESD5V0S2BT, aiee:SOT-23_L2.9-W1.3-P1.90-LS2.4-BR, F.Cu at (74.0, 53.6)
Routing:
- net /ENC_SW: track 108.1 -> 126.7 mm
- net /BTN1: track 76.3 -> 84.0 mm, vias 0 -> 2
- net /BTN2: track 80.6 -> 84.5 mm
- net /BTN3: track 87.0 -> 90.2 mm
- net GND: track 368.3 -> 370.8 mm, vias 17 -> 19
